Commit message: 4444

File: cartographer_ros/cartographer_ros/urdf/my_backpack_2d_sim.urdf (robot description, URDF)
Before this commit: robot cartographer_backpack_2d, 4 links, 3 joints
Joints:
- joint imu_link_joint: parent base_link -> ugv_link
- joint ugv_link_joint: origin xyz=0 0 2 rpy=0. 0 0 -> xyz=0 0 0 rpy=0. 0 0
