Commit message: 22222

File: cartographer_ros/cartographer_ros/urdf/my_backpack_2d.urdf (robot description, URDF)
Before this commit: robot cartographer_backpack_2d, 4 links, 3 joints
Links:
- link laser: geometry visual cylinder length=0.3 radius=0.1
- link ugv_link: geometry visual box size=1 0.5 0.2

Commit message: add imu

File: cartographer_ros/cartographer_ros/urdf/my_backpack_2d.urdf (robot description, URDF)
Before this commit: robot cartographer_backpack_2d, 4 links, 3 joints
Joints:
- joint laser_joint: parent base_link -> ugv_link

Commit message: test ;problem: CPU is fully working

File: cartographer_ros/cartographer_ros/urdf/my_backpack_2d.urdf (robot description, URDF)
Before this commit: robot cartographer_backpack_2d, 4 links, 3 joints
Joints:
- joint imu_link_joint: parent base_link -> ugv_link
